Commit message: Break base link stl into multiple due to mujoco limit

File: isaac_ros-dev/src/bringup/description/shogi.urdf (robot description, URDF)
Before this commit: robot Shogi, 7 links, 6 joints
Links:
- link base_link: geometry collision mesh filename=meshes/base_link_part1.STL; collision mesh filename=meshes/base_link_part2.STL

Commit message: Use shogi urdf

File: isaac_ros-dev/src/bringup/description/shogi.urdf (robot description, URDF)
Before this commit: robot Shogi, 7 links, 6 joints
Links:
- removed link Camera_Link
- removed link GPS_Link
- removed link Left_Wheel_Link
- removed link Lidar_Link
- removed link Right_Wheel_Link
- added link base_footprint
- added link gps_footprint, mass 0.0482645385063794; collision mesh filename=package://bringup/description/meshes/GPS_Link.STL; visual mesh filename=package://bringup/description/meshes/GPS_Link.STL
- added link left_wheel_link, mass 2.0571380710288; collision mesh filename=package://bringup/description/meshes/Left_Wheel_Link.STL; visual mesh filename=package://bringup/description/meshes/Left_Wheel_Link.STL
- added link lidar_footprint, mass 0.762010740793691; collision mesh filename=package://bringup/description/meshes/Lidar_Link.STL; visual mesh filename=package://bringup/description/meshes/Lidar_Link.STL
- added link right_wheel_link, mass 2.0571380823331; collision mesh filename=package://bringup/description/meshes/Right_Wheel_Link.STL; visual mesh filename=package://bringup/description/meshes/Right_Wheel_Link.STL
- added link zed_camera_link, mass 0.170322721037669; collision mesh filename=package://bringup/description/meshes/Camera_Link.STL; visual mesh filename=package://bringup/description/meshes/Camera_Link.STL
- link Caster_link: geometry collision mesh filename=package://bringup/description/meshes/Caster_link.STL; visual mesh filename=package://bringup/description/meshes/Caster_link.STL
- link base_link: geometry collision mesh filename=package://bringup/description/meshes/base_link.STL; visual mesh filename=package://bringup/description/meshes/base_link.STL
Joints:
- added joint base_joint: type fixed, parent base_link, child base_footprint, origin xyz=0 0 0 rpy=0 0 0
- joint Camera: child Camera_Link -> zed_camera_link
- joint GPS: child GPS_Link -> gps_footprint
- joint Left_Wheel: child Left_Wheel_Link -> left_wheel_link
- joint Lidar: child Lidar_Link -> lidar_footprint
- joint Right_Wheel: child Right_Wheel_Link -> right_wheel_link

Commit message: Remove mesh refs

File: isaac_ros-dev/src/bringup/description/shogi.urdf (robot description, URDF)
Before this commit: robot Shogi, 8 links, 7 joints
Links:
- link Caster_link: geometry 
- link base_link: geometry 
- link gps_footprint: geometry 
- link left_wheel_link: geometry 
- link lidar_footprint: geometry 
- link right_wheel_link: geometry 
- link zed_camera_link: geometry 

Commit message: Refactor urdf

File: isaac_ros-dev/src/bringup/description/shogi.urdf (robot description, URDF)
Before this commit: robot Shogi, 8 links, 7 joints
Links:
- link Caster_link: mass 1.38253428199265 -> None; geometry visual mesh filename=package://bringup/description/meshes/Caster_link.STL
- link base_link: mass 24.349 -> None; geometry visual mesh filename=package://bringup/description/meshes/base_link.STL
- link gps_footprint: mass 0.0482645385063794 -> None; geometry visual mesh filename=package://bringup/description/meshes/GPS_Link.STL
- link left_wheel_link: mass 2.0571380710288 -> None; geometry visual mesh filename=package://bringup/description/meshes/Left_Wheel_Link.STL
- link lidar_footprint: mass 0.762010740793691 -> None; geometry visual mesh filename=package://bringup/description/meshes/Lidar_Link.STL
- link right_wheel_link: mass 2.0571380823331 -> None; geometry visual mesh filename=package://bringup/description/meshes/Right_Wheel_Link.STL
- link zed_camera_link: mass 0.170322721037669 -> None; geometry visual mesh filename=package://bringup/description/meshes/Camera_Link.STL
Joints:
- joint Camera: axis 0 0 0 -> (none); origin xyz=0.78801 -2.3703 0.65142 rpy=0.34907 0 0 -> xyz=0.657600 0.009075 0.307230 rpy=0.349070 0 1.570796
- joint Caster: axis 0 0 1 -> (none); limit lower=0 upper=0 effort=0 velocity=0 -> (none); origin xyz=0.77814 -2.2897 0.30331 rpy=1.5708 0 3.1416 -> xyz=0.577000 -0.000795 -0.040880 rpy=1.570800 0 -1.570789; type revolute -> fixed
- joint GPS: axis 0 0 0 -> (none); origin xyz=0.77883 -1.5005 1.0058 rpy=1.5708 0 0 -> xyz=-0.212200 -0.000105 0.661610 rpy=1.570800 0 1.570796
- joint Left_Wheel: axis 1 0 0 -> (none); limit lower=0 upper=0 effort=0 velocity=0 -> (none); origin xyz=0.37276 -1.7127 0.34419 rpy=1.7398 0 0 -> xyz=0 0.361630 0 rpy=1.739800 0 1.570796; type revolute -> fixed
- joint Lidar: axis 0 0 0 -> (none); origin xyz=0.77904 -2.3725 0.54987 rpy=-1.5708 0 0 -> xyz=0.659800 0.000105 0.205680 rpy=-1.570800 0 1.570796
- joint Right_Wheel: axis 1 0 0 -> (none); limit lower=0 upper=0 effort=0 velocity=0 -> (none); origin xyz=0.37276 -1.7127 0.34419 rpy=2.7498 0 -3.1416 -> xyz=0 -0.361630 0 rpy=2.749800 0 -1.570804; type revolute -> fixed
- joint base_joint: origin xyz=0 0 0 rpy=0 0 0 -> xyz=0 0 -0.113030 rpy=0 0 0

Commit message: Rotate lidar

File: isaac_ros-dev/src/bringup/description/shogi.urdf (robot description, URDF)
Before this commit: robot Shogi, 8 links, 7 joints
Joints:
- joint Camera: origin xyz=0.657600 0.009075 0.307230 rpy=0.349070 0 1.570796 -> xyz=0.657600 0.009075 0.307230 rpy=0 0.349070 0
- joint Lidar: origin xyz=0.659800 0.000105 0.205680 rpy=-1.570800 0 1.570796 -> xyz=0.659800 0.000105 0.205680 rpy=-3.141593 -0.000004 0

Commit message: Rotate gps and caster

File: isaac_ros-dev/src/bringup/description/shogi.urdf (robot description, URDF)
Before this commit: robot Shogi, 8 links, 7 joints
Joints:
- joint Caster: origin xyz=0.577000 -0.000795 -0.040880 rpy=1.570800 0 -1.570789 -> xyz=0.577000 -0.000795 -0.040880 rpy=0 -0.000004 0.000007
- joint GPS: origin xyz=-0.212200 -0.000105 0.661610 rpy=1.570800 0 1.570796 -> xyz=-0.212200 -0.000105 0.661610 rpy=1.570796 0.000004 0

Commit message: Rotate gps

File: isaac_ros-dev/src/bringup/description/shogi.urdf (robot description, URDF)
Before this commit: robot Shogi, 8 links, 7 joints
Joints:
- joint GPS: origin xyz=-0.212200 -0.000105 0.661610 rpy=1.570796 0.000004 0 -> xyz=-0.212200 -0.000105 0.661610 rpy=0 0.000004 0

Commit message: fix(urdf): make wheel joints continuous in shogi model
Agent-Logs-Url: https://github.com/KazakhStallion/AutoNav_25-26/sessions/ee117ab0-3a97-453f-abe8-fb6ab6c4630c

Co-authored-by: blobspire <20517406+blobspire@users.noreply.github.com>

File: isaac_ros-dev/src/bringup/description/shogi.urdf (robot description, URDF)
Before this commit: robot Shogi, 8 links, 7 joints
Joints:
- joint Left_Wheel: axis (none) -> 1 0 0; type fixed -> continuous
- joint Right_Wheel: axis (none) -> 1 0 0; type fixed -> continuous

Commit message: Having the NAV2 path spawn from the robot center.

File: isaac_ros-dev/src/bringup/description/shogi.urdf (robot description, URDF)
Before this commit: robot Shogi, 8 links, 7 joints
Links:
- added link nav_center
Joints:
- added joint nav_center_joint: type fixed, parent base_link, child nav_center, origin xyz=0.225 0 0 rpy=0 0 0
