Commit message: feat(bringup): sim-complete shogi.urdf (inertials + gazebo + articulated caster)
Makes shogi.urdf a single sim-complete source of truth so autonav_sim can
spawn it into Gazebo Fortress (previously the sim baked a separate SDF robot
into the world). Adds per-link <inertial>, <collision>, <gazebo> (DiffDrive
plugin, ZED rgbd sensor, wheel/caster friction) and articulates the caster
(fixed -> continuous swivel + caster_wheel_link roll). All functional frames
byte-identical (structural guardrail PASS); added blocks are inert outside
Gazebo. Values ported verbatim from autonav_sim's prior baked world SDF.

VM-verified: converts with no link drops (5 links/4 joints), spawns clean (no
PoseRelativeToGraph), diff-drive publishes /model/shogi/odometry and the robot
drives on /cmd_vel_gazebo.

File: isaac_ros-dev/src/bringup/description/shogi.urdf (robot description, URDF)
Before this commit: robot Shogi, 9 links, 8 joints
Links:
- added link caster_wheel_link, mass 0.35; collision cylinder length=0.064 radius=0.075
- link Caster_link: mass None -> 0.45
- link base_link: mass None -> 48.2703; geometry collision box size=1.09 0.82 0.26; visual mesh filename=package://bringup/description/meshes/base_link.STL
- link left_wheel_link: mass None -> 2.0; geometry collision cylinder length=0.1 radius=0.12946; visual mesh filename=package://bringup/description/meshes/Left_Wheel_Link.STL
- link right_wheel_link: mass None -> 2.0; geometry collision cylinder length=0.1 radius=0.12946; visual mesh filename=package://bringup/description/meshes/Right_Wheel_Link.STL
Joints:
- added joint Caster_Wheel_Roll: type continuous, parent Caster_link, child caster_wheel_link, origin xyz=-0.045000 0 -0.013580 rpy=0 0 0, axis 0 1 0
- joint Caster: axis (none) -> 0 0 1; type fixed -> continuous

Commit message: fix(bringup): reverse Right_Wheel drive axis so the diff-drive drives
Fresh-eyes review caught a CRITICAL sim bug: the Left/Right wheel joints shared
axis '1 0 0' but their origins have opposite-signed yaw, giving ANTIPARALLEL
world spin axes. Gazebo DiffDrive assumes parallel axes, so 'forward' spun the
robot in place and 'rotate' drove it straight. The sim's dead-reckoned
/model/shogi/odometry masked this (it reported forward motion while ground-truth
showed a spin). Reversing Right_Wheel to '-1 0 0' makes both spin axes +Y.
Ground-truth verified: forward -> 2.12 m straight (yaw 0); rotate -> in place.
INERT on the real robot (continuous wheel joints fed q=0 by joint_state_publisher;
at q=0 the TF equals the joint origin regardless of axis sign).

File: isaac_ros-dev/src/bringup/description/shogi.urdf (robot description, URDF)
Before this commit: robot Shogi, 10 links, 9 joints
Joints:
- joint Right_Wheel: axis 1 0 0 -> -1 0 0

Commit message: fix(bringup): rebuild caster from primitives so it renders correctly
Visual inspection in the sim (thanks to running it) caught that the
Caster_link.STL mesh combines the fork AND wheel as one rigid piece. On the
articulated caster (swivel + roll) that rendered as a detached/floating wheel
with the bracket perpendicular, and destabilized the front so the robot tipped.
Rebuilt the caster from primitives (mount/pin cylinders + fork boxes on
Caster_link; a wheel cylinder VISUAL on the rolling caster_wheel_link), verbatim
from the prior baked-SDF caster. VM-verified: renders as a proper upright wheel;
robot drives straight and stays level (base_link RPY 0,0,0, no tipping).

File: isaac_ros-dev/src/bringup/description/shogi.urdf (robot description, URDF)
Before this commit: robot Shogi, 10 links, 9 joints
Links:
- link Caster_link: geometry visual box size=0.036 0.016 0.15; visual box size=0.036 0.016 0.15
- link caster_wheel_link: geometry collision cylinder length=0.064 radius=0.075; visual cylinder length=0.064 radius=0.075
